Commit message: unable to teleop. ackerman introduced

File: qcar_initial/urdf/qcar_model.xacro (robot description, xacro)
@@ -25,9 +25,9 @@
         </inertial>
     </link>
-    <joint name="body_lidar_joint" type="continuous">
-        <parent link="base" />
-        <child link="lidar" />
-        <origin rpy="0 0 0" xyz="-0.01227 -0.00045 0.16152" />
-        <axis xyz="0 0 1" />
+    <joint name="body_lidar_joint" type="fixed">
+        <parent link="base"/>
+        <child link="lidar"/>
+        <origin rpy="0 0 0" xyz="-0.01227 -0.00045 0.16152"/>
+        <axis xyz="0 0 1"/>
     </joint>
     <link name="lidar">
@@ -172,10 +172,10 @@
         <parent link="base" />
         <child link="wheelrl" />
-        <origin rpy="0 0 3.14" xyz="-0.12765 0.05610 0.03338" />
+        <origin rpy="0 0 0" xyz="-0.12765 0.05610 0.03338" />
         <axis xyz="0 1 0" />
     </joint>
     <link name="wheelrl">
         <visual>
-            <origin rpy="0 0 0" xyz="0 0 0" />
+            <origin rpy="0 0 3.14" xyz="0 0 0" />
             <geometry>
                 <mesh filename="package://qcar_initial/models/qcar/QCarWheel.stl"
@@ -185,5 +185,5 @@
         </visual>
         <collision>
-            <origin rpy="0 0 0" xyz="0 0 0" />
+            <origin rpy="0 0 3.14" xyz="0 0 0" />
             <geometry>
                 <mesh filename="package://qcar_initial/models/qcar/QCarWheel.stl"
@@ -368,8 +368,38 @@
         <maxVel>0.1</maxVel>
     </gazebo>
-    <gazebo>
+    <!-- <gazebo>
         <plugin name="gazebo_ros2_control" filename="libgazebo_ros2_control.so">
             <robotNamespace>/qcar</robotNamespace>
             <parameters>$(find qcar_initial)/config/qcar_controllers.yaml</parameters>
+        </plugin>
+    </gazebo> -->
+    <gazebo>
+        <plugin name="ackermann_drive" filename="libgazebo_ros_ackermann_drive.so">
+            <ros>
+                <remapping>cmd_vel:=/cmd_vel</remapping>
+                <remapping>odom:=/odom</remapping>
+            </ros>
+            <!-- Front wheel ROTATION joints (not the steering hubs) -->
+            <front_left_joint>hubfl_wheelfl_joint</front_left_joint>
+            <front_right_joint>hubfr_wheelfr_joint</front_right_joint>
+            <!-- Drive joints (rear wheels) -->
+            <rear_left_joint>base_wheelrl_joint</rear_left_joint>
+            <rear_right_joint>base_wheelrr_joint</rear_right_joint>
+            <!-- Steering hinge joints -->
+            <left_steering_joint>base_hubfl_joint</left_steering_joint>
+            <right_steering_joint>base_hubfr_joint</right_steering_joint>
+            <kingpin_width>0.1122</kingpin_width>       <!-- 2 × 0.05590 front track -->
+            <wheelbase>0.25725</wheelbase>              <!-- 0.12960 + 0.12765 -->
+            <wheel_radius>0.0335</wheel_radius>         <!-- verify against STL -->
+            <max_steer>0.5236</max_steer>              <!-- matches URDF limit (30°) -->
+            <max_speed>2.0</max_speed>
+            <left_steering_pid_gain>10 0 0.5</left_steering_pid_gain>
+            <right_steering_pid_gain>10 0 0.5</right_steering_pid_gain>
+            <linear_velocity_pid_gain>10 0 0.5</linear_velocity_pid_gain>
+            <publish_odom>true</publish_odom>
+            <publish_odom_tf>true</publish_odom_tf>
+            <publish_wheel_tf>true</publish_wheel_tf>
+            <odometry_frame>odom</odometry_frame>
+            <robot_base_frame>base</robot_base_frame>
         </plugin>
     </gazebo>
@@ -409,5 +439,5 @@
         </sensor>
     </gazebo>
-    <ros2_control name="qcar" type="system">
+    <!-- <ros2_control name="qcar" type="system">
         <hardware>
             <plugin>gazebo_ros2_control/GazeboSystem</plugin>
@@ -433,4 +463,4 @@
             <state_interface name="velocity" />
         </joint>
-    </ros2_control>
+    </ros2_control> -->
 </robot>

Commit message: reverted to drive control. nav2 up and running. not accurate

File: qcar_initial/urdf/qcar_model.xacro (robot description, xacro)
@@ -172,10 +172,10 @@
         <parent link="base" />
         <child link="wheelrl" />
-        <origin rpy="0 0 0" xyz="-0.12765 0.05610 0.03338" />
+        <origin rpy="0 0 3.14" xyz="-0.12765 0.05610 0.03338" />
         <axis xyz="0 1 0" />
     </joint>
     <link name="wheelrl">
         <visual>
-            <origin rpy="0 0 3.14" xyz="0 0 0" />
+            <origin rpy="0 0 0" xyz="0 0 0" />
             <geometry>
                 <mesh filename="package://qcar_initial/models/qcar/QCarWheel.stl"
@@ -185,5 +185,5 @@
         </visual>
         <collision>
-            <origin rpy="0 0 3.14" xyz="0 0 0" />
+            <origin rpy="0 0 0" xyz="0 0 0" />
             <geometry>
                 <mesh filename="package://qcar_initial/models/qcar/QCarWheel.stl"
@@ -352,5 +352,5 @@
         </sensor>
     </gazebo>
-    <gazebo reference="wheelrl">
+    <!-- <gazebo reference="wheelrl">
         <mu1>1.0</mu1>
         <mu2>1.0</mu2>
@@ -367,12 +367,12 @@
         <minDepth>0.001</minDepth>
         <maxVel>0.1</maxVel>
-    </gazebo>
-    <!-- <gazebo>
+    </gazebo> -->
+    <gazebo>
         <plugin name="gazebo_ros2_control" filename="libgazebo_ros2_control.so">
             <robotNamespace>/qcar</robotNamespace>
             <parameters>$(find qcar_initial)/config/qcar_controllers.yaml</parameters>
         </plugin>
-    </gazebo> -->
-    <gazebo>
+    </gazebo>
+    <!-- <gazebo>
         <plugin name="ackermann_drive" filename="libgazebo_ros_ackermann_drive.so">
             <ros>
@@ -380,21 +380,25 @@
                 <remapping>odom:=/odom</remapping>
             </ros>
-            <!-- Front wheel ROTATION joints (not the steering hubs) -->
+            <update_rate>100.0</update_rate>
+            Front wheel ROTATION joints (not the steering hubs)
             <front_left_joint>hubfl_wheelfl_joint</front_left_joint>
             <front_right_joint>hubfr_wheelfr_joint</front_right_joint>
-            <!-- Drive joints (rear wheels) -->
+            Drive joints (rear wheels)
             <rear_left_joint>base_wheelrl_joint</rear_left_joint>
             <rear_right_joint>base_wheelrr_joint</rear_right_joint>
-            <!-- Steering hinge joints -->
+            Steering hinge joints
             <left_steering_joint>base_hubfl_joint</left_steering_joint>
             <right_steering_joint>base_hubfr_joint</right_steering_joint>
-            <kingpin_width>0.1122</kingpin_width>       <!-- 2 × 0.05590 front track -->
-            <wheelbase>0.25725</wheelbase>              <!-- 0.12960 + 0.12765 -->
-            <wheel_radius>0.0335</wheel_radius>         <!-- verify against STL -->
-            <max_steer>0.5236</max_steer>              <!-- matches URDF limit (30°) -->
+            <kingpin_width>0.1122</kingpin_width>       2 × 0.05590 front track
+            <wheelbase>0.25725</wheelbase>              0.12960 + 0.12765
+            <wheel_radius>0.0335</wheel_radius>         verify against STL
+            <max_steer>0.5236</max_steer>              matches URDF limit (30°)
             <max_speed>2.0</max_speed>
             <left_steering_pid_gain>10 0 0.5</left_steering_pid_gain>
+            <left_steering_i_range>0 0</left_steering_i_range>
             <right_steering_pid_gain>10 0 0.5</right_steering_pid_gain>
+            <right_steering_i_range>0 0</right_steering_i_range>
             <linear_velocity_pid_gain>10 0 0.5</linear_velocity_pid_gain>
+            <linear_velocity_i_range>0 0</linear_velocity_i_range>
             <publish_odom>true</publish_odom>
             <publish_odom_tf>true</publish_odom_tf>
@@ -403,5 +407,5 @@
             <robot_base_frame>base</robot_base_frame>
         </plugin>
-    </gazebo>
+    </gazebo> -->
     <!-- LiDAR Sensor -->
     <gazebo reference="lidar">
@@ -439,5 +443,5 @@
         </sensor>
     </gazebo>
-    <!-- <ros2_control name="qcar" type="system">
+    <ros2_control name="qcar" type="system">
         <hardware>
             <plugin>gazebo_ros2_control/GazeboSystem</plugin>
@@ -463,4 +467,4 @@
             <state_interface name="velocity" />
         </joint>
-    </ros2_control> -->
+    </ros2_control>
 </robot>
