Commit message: updated and added to initial

File: qcar_initial/urdf/qcar_model.xacro (robot description, xacro)
@@ -2,5 +2,4 @@
 <robot name="QCar" xmlns:xacro="http://www.ros.org/wiki/xacro">
     <xacro:include filename="$(find qcar_initial)/urdf/materials.xacro" />
-    <xacro:include filename="$(find realsense2_description)/urdf/_d435.urdf.xacro" />
     <link name="base">
         <visual>
@@ -21,6 +20,6 @@
         <inertial>
             <origin rpy="0 0 0" xyz="0 0 0" />
-            <mass value="0.1" />
-            <inertia ixx="0.001" ixy="0" ixz="0" iyy="0.001" iyz="0" izz="0.001" />
+            <mass value="2.4" />
+            <inertia ixx="0.009543" ixy="0" ixz="0" iyy="0.038083" iyz="0" izz="0.038274" />
         </inertial>
     </link>
@@ -49,6 +48,6 @@
         <inertial>
             <origin rpy="0 0 0" xyz="0 0 0" />
-            <mass value="0.1" />
-            <inertia ixx="0.001" ixy="0" ixz="0" iyy="0.001" iyz="0" izz="0.001" />
+            <mass value="0.15" />
+            <inertia ixx="0.0000724" ixy="0" ixz="0" iyy="0.0000724" iyz="0" izz="0.000133" />
         </inertial>
     </link>
@@ -79,6 +78,6 @@
         <inertial>
             <origin rpy="0 0 0" xyz="0 0 0" />
-            <mass value="0.1" />
-            <inertia ixx="0.001" ixy="0" ixz="0" iyy="0.001" iyz="0" izz="0.001" />
+            <mass value="0.05" />
+            <inertia ixx="0.00000925" ixy="0" ixz="0" iyy="0.0000131" iyz="0" izz="0.00000843" />
         </inertial>
     </link>
@@ -109,6 +108,6 @@
         <inertial>
             <origin rpy="0 0 0" xyz="0 0 0" />
-            <mass value="0.1" />
-            <inertia ixx="0.001" ixy="0" ixz="0" iyy="0.001" iyz="0" izz="0.001" />
+            <mass value="0.05" />
+            <inertia ixx="0.00000925" ixy="0" ixz="0" iyy="0.0000131" iyz="0" izz="0.00000843" />
         </inertial>
     </link>
@@ -137,6 +136,6 @@
         <inertial>
             <origin rpy="0 0 0" xyz="0 0 0" />
-            <mass value="0.1" />
-            <inertia ixx="0.001" ixy="0" ixz="0" iyy="0.001" iyz="0" izz="0.001" />
+            <mass value="0.2" />
+            <inertia ixx="0.0000645" ixy="0" ixz="0" iyy="0.0001089" iyz="0" izz="0.0000645" />
         </inertial>
     </link>
@@ -165,6 +164,6 @@
         <inertial>
             <origin rpy="0 0 0" xyz="0 0 0" />
-            <mass value="0.1" />
-            <inertia ixx="0.001" ixy="0" ixz="0" iyy="0.001" iyz="0" izz="0.001" />
+            <mass value="0.2" />
+            <inertia ixx="0.0000645" ixy="0" ixz="0" iyy="0.0001089" iyz="0" izz="0.0000645" />
         </inertial>
     </link>
@@ -193,6 +192,6 @@
         <inertial>
             <origin rpy="0 0 0" xyz="0 0 0" />
-            <mass value="0.1" />
-            <inertia ixx="0.001" ixy="0" ixz="0" iyy="0.001" iyz="0" izz="0.001" />
+            <mass value="0.2" />
+            <inertia ixx="0.0000645" ixy="0" ixz="0" iyy="0.0001089" iyz="0" izz="0.0000645" />
         </inertial>
     </link>
@@ -221,6 +220,6 @@
         <inertial>
             <origin rpy="0 0 0" xyz="0 0 0" />
-            <mass value="0.1" />
-            <inertia ixx="0.001" ixy="0" ixz="0" iyy="0.001" iyz="0" izz="0.001" />
+            <mass value="0.2" />
+            <inertia ixx="0.0000645" ixy="0" ixz="0" iyy="0.0001089" iyz="0" izz="0.0000645" />
         </inertial>
     </link>
@@ -270,70 +269,4 @@
     </joint>
     <link name="camera_csi_left" />
-    <transmission name="body_lidar_tran">
-        <type>transmission_interface/SimpleTransmission</type>
-        <joint name="body_lidar_joint">
-            <hardwareInterface>hardware_interface/EffortJointInterface</hardwareInterface>
-        </joint>
-        <actuator name="body_lidar_motor">
-            <mechanicalReduction>1</mechanicalReduction>
-        </actuator>
-    </transmission>
-    <transmission name="base_hubfl_tran">
-        <type>transmission_interface/SimpleTransmission</type>
-        <joint name="base_hubfl_joint">
-            <hardwareInterface>hardware_interface/PositionJointInterface</hardwareInterface>
-        </joint>
-        <actuator name="base_hubfl_motor">
-            <mechanicalReduction>1</mechanicalReduction>
-        </actuator>
-    </transmission>
-    <transmission name="base_hubfr_tran">
-        <type>transmission_interface/SimpleTransmission</type>
-        <joint name="base_hubfr_joint">
-            <hardwareInterface>hardware_interface/PositionJointInterface</hardwareInterface>
-        </joint>
-        <actuator name="base_hubfr_motor">
-            <mechanicalReduction>1</mechanicalReduction>
-        </actuator>
-    </transmission>
-    <transmission name="hubfl_wheelfl_tran">
-        <type>transmission_interface/SimpleTransmission</type>
-        <joint name="hubfl_wheelfl_joint">
-            <hardwareInterface>hardware_interface/EffortJointInterface</hardwareInterface>
-        </joint>
-        <actuator name="hubfl_wheelfl_motor">
-            <mechanicalReduction>1</mechanicalReduction>
-        </actuator>
-    </transmission>
-    <transmission name="hubfr_wheelfr_tran">
-        <type>transmission_interface/SimpleTransmission</type>
-        <joint name="hubfr_wheelfr_joint">
-            <hardwareInterface>hardware_interface/EffortJointInterface</hardwareInterface>
-        </joint>
-        <actuator name="hubfr_wheelfr_motor">
-            <mechanicalReduction>1</mechanicalReduction>
-        </actuator>
-    </transmission>
-    <transmission name="base_wheelrl_tran">
-        <type>transmission_interface/SimpleTransmission</type>
-        <joint name="base_wheelrl_joint">
-            <hardwareInterface>hardware_interface/VelocityJointInterface</hardwareInterface>
-        </joint>
-        <actuator name="base_wheelrl_motor">
-            <mechanicalReduction>1</mechanicalReduction>
-        </actuator>
-    </transmission>
-    <transmission name="base_wheelrr_tran">
-        <type>transmission_interface/SimpleTransmission</type>
-        <joint name="base_wheelrr_joint">
-            <hardwareInterface>hardware_interface/VelocityJointInterface</hardwareInterface>
-        </joint>
-        <actuator name="base_wheelrr_motor">
-            <mechanicalReduction>1</mechanicalReduction>
-        </actuator>
-    </transmission>
-    <!-- <xacro:sensor_d435 name="camera" parent="camera_rgb">
-        <origin xyz="0 0 0" rpy="0 0 0" />
-    </xacro:sensor_d435>   -->
     <gazebo reference="camera_csi_front">
         <sensor type="camera" name="front_camera">
@@ -352,60 +285,9 @@
         </sensor>
     </gazebo>
-    <!-- <gazebo reference="wheelrl">
-        <mu1>1.0</mu1>
-        <mu2>1.0</mu2>
-        <kp>500000.0</kp>
-        <kd>10.0</kd>
-        <minDepth>0.001</minDepth>
-        <maxVel>0.1</maxVel>
-    </gazebo>
-    <gazebo reference="wheelrr">
-        <mu1>1.0</mu1>
-        <mu2>1.0</mu2>
-        <kp>500000.0</kp>
-        <kd>10.0</kd>
-        <minDepth>0.001</minDepth>
-        <maxVel>0.1</maxVel>
-    </gazebo> -->
     <gazebo>
         <plugin name="gazebo_ros2_control" filename="libgazebo_ros2_control.so">
-            <robotNamespace>/qcar</robotNamespace>
             <parameters>$(find qcar_initial)/config/qcar_controllers.yaml</parameters>
         </plugin>
     </gazebo>
-    <!-- <gazebo>
-        <plugin name="ackermann_drive" filename="libgazebo_ros_ackermann_drive.so">
-            <ros>
-                <remapping>cmd_vel:=/cmd_vel</remapping>
-                <remapping>odom:=/odom</remapping>
-            </ros>
-            <update_rate>100.0</update_rate>
-            Front wheel ROTATION joints (not the steering hubs)
-            <front_left_joint>hubfl_wheelfl_joint</front_left_joint>
-            <front_right_joint>hubfr_wheelfr_joint</front_right_joint>
-            Drive joints (rear wheels)
-            <rear_left_joint>base_wheelrl_joint</rear_left_joint>
-            <rear_right_joint>base_wheelrr_joint</rear_right_joint>
-            Steering hinge joints
-            <left_steering_joint>base_hubfl_joint</left_steering_joint>
-            <right_steering_joint>base_hubfr_joint</right_steering_joint>
-            <kingpin_width>0.1122</kingpin_width>       2 × 0.05590 front track
-            <wheelbase>0.25725</wheelbase>              0.12960 + 0.12765
-            <wheel_radius>0.0335</wheel_radius>         verify against STL
-            <max_steer>0.5236</max_steer>              matches URDF limit (30°)
-            <max_speed>2.0</max_speed>
-            <left_steering_pid_gain>10 0 0.5</left_steering_pid_gain>
-            <left_steering_i_range>0 0</left_steering_i_range>
-            <right_steering_pid_gain>10 0 0.5</right_steering_pid_gain>
-            <right_steering_i_range>0 0</right_steering_i_range>
-            <linear_velocity_pid_gain>10 0 0.5</linear_velocity_pid_gain>
-            <linear_velocity_i_range>0 0</linear_velocity_i_range>
-            <publish_odom>true</publish_odom>
-            <publish_odom_tf>true</publish_odom_tf>
-            <publish_wheel_tf>true</publish_wheel_tf>
-            <odometry_frame>odom</odometry_frame>
-            <robot_base_frame>base</robot_base_frame>
-        </plugin>
-    </gazebo> -->
     <!-- LiDAR Sensor -->
     <gazebo reference="lidar">
@@ -454,5 +336,5 @@
             <xyz_offset>0 0 0</xyz_offset>
             <rpy_offset>0 0 0</rpy_offset>
-            <gaussian_noise>0.0</gaussian_noise>
+            <gaussian_noise>0.01</gaussian_noise>
         </plugin>
     </gazebo>
