Commit message: modified qcar_updated package with ackerman steering - lidar issue exist, robot drifts

File: qcar_updated/urdf/qcar_model.xacro (robot description, xacro)
@@ -172,5 +172,8 @@
         <child link="wheelrl" />
         <origin rpy="0 0 3.14" xyz="-0.12765 0.05610 0.03338" />
-        <axis xyz="0 1 0" />
+        <!-- axis negated to compensate for the 180deg yaw above (mesh mirror) -
+             without this the left wheel spins opposite the right wheel for the
+             same signed velocity command -->
+        <axis xyz="0 -1 0" />
     </joint>
     <link name="wheelrl">
@@ -325,18 +328,4 @@
         </sensor>
     </gazebo>
-    <!-- Ground truth odometry from Gazebo physics -->
-    <gazebo>
-        <plugin name="gazebo_ros_p3d" filename="libgazebo_ros_p3d.so">
-            <ros>
-                <remapping>odom:=/odom</remapping>
-            </ros>
-            <body_name>base</body_name>
-            <frame_name>world</frame_name>
-            <update_rate>30</update_rate>
-            <xyz_offset>0 0 0</xyz_offset>
-            <rpy_offset>0 0 0</rpy_offset>
-            <gaussian_noise>0.01</gaussian_noise>
-        </plugin>
-    </gazebo>
     <ros2_control name="qcar" type="system">
         <hardware>
