Commit message: multiple corrections made: initial is working with ros2 control and updated with ackermann. 2 other packages not working

File: qcar_ackermann/urdf/qcar_model.xacro (robot description, xacro)
@@ -1,10 +1,10 @@
 <?xml version='1.0'?>
 <robot name="QCar" xmlns:xacro="http://www.ros.org/wiki/xacro">
-  <xacro:include filename="$(find qcar_updated)/urdf/materials.xacro" />
+    <xacro:include filename="$(find qcar_ackermann)/urdf/materials.xacro" />
     <link name="base">
         <visual>
             <origin rpy="0 0 0" xyz="0 0 0" />
             <geometry>
-                <mesh filename="package://qcar_updated/models/qcar/QCarBody.stl"
+                <mesh filename="package://qcar_ackermann/models/qcar/QCarBody.stl"
                     scale="0.001 0.001 0.001" />
             </geometry>
@@ -14,5 +14,5 @@
             <origin rpy="0 0 0" xyz="0 0 0" />
             <geometry>
-                <mesh filename="package://qcar_updated/models/qcar/QCarBody.stl"
+                <mesh filename="package://qcar_ackermann/models/qcar/QCarBody.stl"
                     scale="0.001 0.001 0.001" />
             </geometry>
@@ -34,5 +34,5 @@
             <origin rpy="0 0 0" xyz="0 0 0" />
             <geometry>
-                <mesh filename="package://qcar_updated/models/qcar/QCarLidar.stl"
+                <mesh filename="package://qcar_ackermann/models/qcar/QCarLidar.stl"
                     scale="0.001 0.001 0.001" />
             </geometry>
@@ -42,5 +42,5 @@
             <origin rpy="0 0 0" xyz="0 0 0" />
             <geometry>
-                <mesh filename="package://qcar_updated/models/qcar/QCarLidar.stl"
+                <mesh filename="package://qcar_ackermann/models/qcar/QCarLidar.stl"
                     scale="0.001 0.001 0.001" />
             </geometry>
@@ -64,5 +64,5 @@
             <origin rpy="0 0 0" xyz="0 0 0" />
             <geometry>
-                <mesh filename="package://qcar_updated/models/qcar/QCarSteeringHubL.stl"
+                <mesh filename="package://qcar_ackermann/models/qcar/QCarSteeringHubL.stl"
                     scale="0.001 0.001 0.001" />
             </geometry>
@@ -72,5 +72,5 @@
             <origin rpy="0 0 0" xyz="0 0 0" />
             <geometry>
-                <mesh filename="package://qcar_updated/models/qcar/QCarSteeringHubL.stl"
+                <mesh filename="package://qcar_ackermann/models/qcar/QCarSteeringHubL.stl"
                     scale="0.001 0.001 0.001" />
             </geometry>
@@ -94,5 +94,5 @@
             <origin rpy="0 0 0" xyz="0 0 0" />
             <geometry>
-                <mesh filename="package://qcar_updated/models/qcar/QCarSteeringHubR.stl"
+                <mesh filename="package://qcar_ackermann/models/qcar/QCarSteeringHubR.stl"
                     scale="0.001 0.001 0.001" />
             </geometry>
@@ -102,5 +102,5 @@
             <origin rpy="0 0 0" xyz="0 0 0" />
             <geometry>
-                <mesh filename="package://qcar_updated/models/qcar/QCarSteeringHubR.stl"
+                <mesh filename="package://qcar_ackermann/models/qcar/QCarSteeringHubR.stl"
                     scale="0.001 0.001 0.001" />
             </geometry>
@@ -116,7 +116,5 @@
         <child link="wheelfl" />
         <origin rpy="0 0 3.14" xyz="0 0 0" />
-        <!-- axis negated to compensate for the 180deg yaw above (mesh mirror) -
-             without this the left wheel spins opposite the right wheel -->
-        <axis xyz="0 -1 0" />
+        <axis xyz="0 1 0" />
     </joint>
     <link name="wheelfl">
@@ -124,18 +122,14 @@
             <origin rpy="0 0 0" xyz="0 0 0" />
             <geometry>
-                <mesh filename="package://qcar_updated/models/qcar/QCarWheel.stl"
+                <mesh filename="package://qcar_ackermann/models/qcar/QCarWheel.stl"
                     scale="0.001 0.001 0.001" />
             </geometry>
             <material name="red" />
         </visual>
-        <!-- collision is a cylinder, not the visual mesh - the ackermann drive
-             plugin's wheel-radius auto-detection only supports cylinder/sphere
-             collisions; with a mesh it silently reads radius=0 and poisons the
-             velocity PID. Radius is 3mm over the mesh's actual 0.033m to
-             guarantee real ground penetration/contact force. -->
-        <collision>
-            <origin rpy="1.5708 0 0" xyz="0 0 0" />
-            <geometry>
-                <cylinder radius="0.036" length="0.0245" />
+        <collision>
+            <origin rpy="0 0 0" xyz="0 0 0" />
+            <geometry>
+                <mesh filename="package://qcar_ackermann/models/qcar/QCarWheel.stl"
+                    scale="0.001 0.001 0.001" />
             </geometry>
         </collision>
@@ -143,5 +137,5 @@
             <origin rpy="0 0 0" xyz="0 0 0" />
             <mass value="0.2" />
-            <inertia ixx="0.0012" ixy="0" ixz="0" iyy="0.0022" iyz="0" izz="0.0012" />
+            <inertia ixx="0.0000645" ixy="0" ixz="0" iyy="0.0001089" iyz="0" izz="0.0000645" />
         </inertial>
     </link>
@@ -156,5 +150,5 @@
             <origin rpy="0 0 0" xyz="0 0 0" />
             <geometry>
-                <mesh filename="package://qcar_updated/models/qcar/QCarWheel.stl"
+                <mesh filename="package://qcar_ackermann/models/qcar/QCarWheel.stl"
                     scale="0.001 0.001 0.001" />
             </geometry>
@@ -162,7 +156,8 @@
         </visual>
         <collision>
-            <origin rpy="1.5708 0 0" xyz="0 0 0" />
-            <geometry>
-                <cylinder radius="0.036" length="0.0245" />
+            <origin rpy="0 0 0" xyz="0 0 0" />
+            <geometry>
+                <mesh filename="package://qcar_ackermann/models/qcar/QCarWheel.stl"
+                    scale="0.001 0.001 0.001" />
             </geometry>
         </collision>
@@ -170,5 +165,5 @@
             <origin rpy="0 0 0" xyz="0 0 0" />
             <mass value="0.2" />
-            <inertia ixx="0.0012" ixy="0" ixz="0" iyy="0.0022" iyz="0" izz="0.0012" />
+            <inertia ixx="0.0000645" ixy="0" ixz="0" iyy="0.0001089" iyz="0" izz="0.0000645" />
         </inertial>
     </link>
@@ -177,8 +172,5 @@
         <child link="wheelrl" />
         <origin rpy="0 0 3.14" xyz="-0.12765 0.05610 0.03338" />
-        <!-- axis negated to compensate for the 180deg yaw above (mesh mirror) -
-             without this the left wheel spins opposite the right wheel for the
-             same signed velocity command -->
-        <axis xyz="0 -1 0" />
+        <axis xyz="0 1 0" />
     </joint>
     <link name="wheelrl">
@@ -186,5 +178,5 @@
             <origin rpy="0 0 0" xyz="0 0 0" />
             <geometry>
-                <mesh filename="package://qcar_updated/models/qcar/QCarWheel.stl"
+                <mesh filename="package://qcar_ackermann/models/qcar/QCarWheel.stl"
                     scale="0.001 0.001 0.001" />
             </geometry>
@@ -192,7 +184,8 @@
         </visual>
         <collision>
-            <origin rpy="1.5708 0 0" xyz="0 0 0" />
-            <geometry>
-                <cylinder radius="0.036" length="0.0245" />
+            <origin rpy="0 0 0" xyz="0 0 0" />
+            <geometry>
+                <mesh filename="package://qcar_ackermann/models/qcar/QCarWheel.stl"
+                    scale="0.001 0.001 0.001" />
             </geometry>
         </collision>
@@ -200,5 +193,5 @@
             <origin rpy="0 0 0" xyz="0 0 0" />
             <mass value="0.2" />
-            <inertia ixx="0.0012" ixy="0" ixz="0" iyy="0.0022" iyz="0" izz="0.0012" />
+            <inertia ixx="0.0000645" ixy="0" ixz="0" iyy="0.0001089" iyz="0" izz="0.0000645" />
         </inertial>
     </link>
@@ -213,5 +206,5 @@
             <origin rpy="0 0 0" xyz="0 0 0" />
             <geometry>
-                <mesh filename="package://qcar_updated/models/qcar/QCarWheel.stl"
+                <mesh filename="package://qcar_ackermann/models/qcar/QCarWheel.stl"
                     scale="0.001 0.001 0.001" />
             </geometry>
@@ -219,7 +212,8 @@
         </visual>
         <collision>
-            <origin rpy="1.5708 0 0" xyz="0 0 0" />
-            <geometry>
-                <cylinder radius="0.036" length="0.0245" />
+            <origin rpy="0 0 0" xyz="0 0 0" />
+            <geometry>
+                <mesh filename="package://qcar_ackermann/models/qcar/QCarWheel.stl"
+                    scale="0.001 0.001 0.001" />
             </geometry>
         </collision>
@@ -227,25 +221,7 @@
             <origin rpy="0 0 0" xyz="0 0 0" />
             <mass value="0.2" />
-            <inertia ixx="0.0012" ixy="0" ixz="0" iyy="0.0022" iyz="0" izz="0.0012" />
-        </inertial>
-    </link>
-    <!-- wheel-ground friction - without this the wheels spin freely with 100%
-         slip and the chassis never translates, regardless of PID gains -->
-    <gazebo reference="wheelfl">
-        <mu1>1.0</mu1>
-        <mu2>1.0</mu2>
-    </gazebo>
-    <gazebo reference="wheelfr">
-        <mu1>1.0</mu1>
-        <mu2>1.0</mu2>
-    </gazebo>
-    <gazebo reference="wheelrl">
-        <mu1>1.0</mu1>
-        <mu2>1.0</mu2>
-    </gazebo>
-    <gazebo reference="wheelrr">
-        <mu1>1.0</mu1>
-        <mu2>1.0</mu2>
-    </gazebo>
+            <inertia ixx="0.0000645" ixy="0" ixz="0" iyy="0.0001089" iyz="0" izz="0.0000645" />
+        </inertial>
+    </link>
     <joint name="camera_rgb_joint" type="fixed">
         <!-- <axis xyz="0 1 0" /> -->
@@ -309,46 +285,9 @@
         </sensor>
     </gazebo>
-    <gazebo>
-        <plugin name="gazebo_ros_ackermann_drive" filename="libgazebo_ros_ackermann_drive.so">
-            <update_rate>100.0</update_rate>
-            <!-- front wheel spin joints (child of the steering hubs) -->
-            <front_left_joint>hubfl_wheelfl_joint</front_left_joint>
-            <front_right_joint>hubfr_wheelfr_joint</front_right_joint>
-            <!-- rear drive wheel joints -->
-            <rear_left_joint>base_wheelrl_joint</rear_left_joint>
-            <rear_right_joint>base_wheelrr_joint</rear_right_joint>
-            <!-- front hub steering (yaw) joints -->
-            <left_steering_joint>base_hubfl_joint</left_steering_joint>
-            <right_steering_joint>base_hubfr_joint</right_steering_joint>
-            <!-- wheelbase/track/wheel radius are auto-computed by the plugin
-                 from the joints' actual poses/collision geometry in this URDF -->
-            <!-- Real QCar steering limit: 30 deg -->
-            <max_steer>0.5236</max_steer>
-            <max_speed>20</max_speed>
-            <!-- PID tuning: the upstream demo's gains (1500/1000) were tuned for a
-                 full-size car and are ~1000x too aggressive for this vehicle's wheel
-                 inertia, causing an immediate physics blowup (confirmed by testing).
-                 0.3/0/0.02 steering gain still destabilized the sim (gzserver crash
-                 in Ogre::AxisAlignedBox::setExtents) even with the wheel inertia bump
-                 above - these lower values are confirmed stable. -->
-            <left_steering_pid_gain>0.02 0 0.002</left_steering_pid_gain>
-            <left_steering_i_range>0 0</left_steering_i_range>
-            <right_steering_pid_gain>0.02 0 0.002</right_steering_pid_gain>
-            <right_steering_i_range>0 0</right_steering_i_range>
-            <linear_velocity_pid_gain>0.3 0 0.005</linear_velocity_pid_gain>
-            <linear_velocity_i_range>0 0</linear_velocity_i_range>
-            <publish_odom>true</publish_odom>
-            <publish_odom_tf>true</publish_odom_tf>
-            <publish_wheel_tf>true</publish_wheel_tf>
-            <publish_distance>false</publish_distance>
-            <odometry_frame>odom</odometry_frame>
-            <robot_base_frame>base</robot_base_frame>
-        </plugin>
-    </gazebo>
     <!-- LiDAR Sensor -->
     <gazebo reference="lidar">
         <sensor type="ray" name="lidar_sensor">
             <pose>0 0 0 0 0 0</pose>
-            <visualize>true</visualize>
+            <visualize>false</visualize>
             <update_rate>10</update_rate>
             <ray>
@@ -381,3 +320,37 @@
         </sensor>
     </gazebo>
-  </robot>
+    <!-- Ackermann drive plugin -->
+    <gazebo>
+        <plugin name="ackermann_drive" filename="libgazebo_ros_ackermann_drive.so">
+            <ros>
+                <namespace></namespace>
+            </ros>
+            <update_rate>100.0</update_rate>
+            <front_left_joint>hubfl_wheelfl_joint</front_left_joint>
+            <front_right_joint>hubfr_wheelfr_joint</front_right_joint>
+            <rear_left_joint>base_wheelrl_joint</rear_left_joint>
+            <rear_right_joint>base_wheelrr_joint</rear_right_joint>
+            <left_steering_joint>base_hubfl_joint</left_steering_joint>
+            <right_steering_joint>base_hubfr_joint</right_steering_joint>
+            <max_steer>0.5236</max_steer>
+            <max_steering_angle>0.5236</max_steering_angle>
+            <max_speed>3.0</max_speed>
+            <left_steering_pid_gain>5 0 0.1</left_steering_pid_gain>
+            <left_steering_i_range>0 0</left_steering_i_range>
+            <right_steering_pid_gain>5 0 0.1</right_steering_pid_gain>
+            <right_steering_i_range>0 0</right_steering_i_range>
+            <linear_velocity_pid_gain>10 0 0.5</linear_velocity_pid_gain>
+            <linear_velocity_i_range>0 0</linear_velocity_i_range>
+            <wheel_base>0.257</wheel_base>
+            <wheel_separation>0.112</wheel_separation>
+            <wheel_diameter>0.066</wheel_diameter>
+            <publish_odom>true</publish_odom>
+            <publish_odom_tf>true</publish_odom_tf>
+            <publish_wheel_tf>true</publish_wheel_tf>
+            <odometry_topic>odom</odometry_topic>
+            <odometry_frame>odom</odometry_frame>
+            <robot_base_frame>base</robot_base_frame>
+            <command_topic>cmd_vel</command_topic>
+        </plugin>
+    </gazebo>
+</robot>
