Commit message: multiple corrections made: initial is working with ros2 control and updated with ackermann. 2 other packages not working

File: qcar_navigation/urdf/qcar2.urdf.xacro (robot description, xacro)
@@ -6,5 +6,5 @@
             <origin rpy="0 0 0" xyz="0 0 0" />
             <geometry>
-                <mesh filename="package://qcar_updated/models/qcar/QCarBody.stl"
+                <mesh filename="file://$(find qcar_navigation)/meshes/QCar2Body.stl"
                     scale="0.001 0.001 0.001" />
             </geometry>
@@ -14,5 +14,5 @@
             <origin rpy="0 0 0" xyz="0 0 0" />
             <geometry>
-                <mesh filename="package://qcar_updated/models/qcar/QCarBody.stl"
+                <mesh filename="file://$(find qcar_navigation)/meshes/QCar2Body.stl"
                     scale="0.001 0.001 0.001" />
             </geometry>
@@ -34,5 +34,5 @@
             <origin rpy="0 0 0" xyz="0 0 0" />
             <geometry>
-                <mesh filename="package://qcar_updated/models/qcar/QCarLidar.stl"
+                <mesh filename="file://$(find qcar_navigation)/meshes/QCar2Lidar.stl"
                     scale="0.001 0.001 0.001" />
             </geometry>
@@ -42,5 +42,5 @@
             <origin rpy="0 0 0" xyz="0 0 0" />
             <geometry>
-                <mesh filename="package://qcar_updated/models/qcar/QCarLidar.stl"
+                <mesh filename="file://$(find qcar_navigation)/meshes/QCar2Lidar.stl"
                     scale="0.001 0.001 0.001" />
             </geometry>
@@ -64,5 +64,5 @@
             <origin rpy="0 0 0" xyz="0 0 0" />
             <geometry>
-                <mesh filename="package://qcar_updated/models/qcar/QCarSteeringHubL.stl"
+                <mesh filename="file://$(find qcar_navigation)/meshes/QCarSteeringHubL.stl"
                     scale="0.001 0.001 0.001" />
             </geometry>
@@ -72,5 +72,5 @@
             <origin rpy="0 0 0" xyz="0 0 0" />
             <geometry>
-                <mesh filename="package://qcar_updated/models/qcar/QCarSteeringHubL.stl"
+                <mesh filename="file://$(find qcar_navigation)/meshes/QCarSteeringHubL.stl"
                     scale="0.001 0.001 0.001" />
             </geometry>
@@ -94,5 +94,5 @@
             <origin rpy="0 0 0" xyz="0 0 0" />
             <geometry>
-                <mesh filename="package://qcar_updated/models/qcar/QCarSteeringHubR.stl"
+                <mesh filename="file://$(find qcar_navigation)/meshes/QCarSteeringHubR.stl"
                     scale="0.001 0.001 0.001" />
             </geometry>
@@ -102,5 +102,5 @@
             <origin rpy="0 0 0" xyz="0 0 0" />
             <geometry>
-                <mesh filename="package://qcar_updated/models/qcar/QCarSteeringHubR.stl"
+                <mesh filename="file://$(find qcar_navigation)/meshes/QCarSteeringHubR.stl"
                     scale="0.001 0.001 0.001" />
             </geometry>
@@ -124,15 +124,16 @@
             <origin rpy="0 0 0" xyz="0 0 0" />
             <geometry>
-                <mesh filename="package://qcar_updated/models/qcar/QCarWheel.stl"
+                <mesh filename="file://$(find qcar_navigation)/meshes/QCarWheel.stl"
                     scale="0.001 0.001 0.001" />
             </geometry>
             <material name="red" />
         </visual>
-        <!-- collision is a cylinder, not the visual mesh - the ackermann drive
-             plugin's wheel-radius auto-detection only supports cylinder/sphere
-             collisions; with a mesh it silently reads radius=0 and poisons the
-             velocity PID. Radius is 3mm over the mesh's actual 0.033m to
-             guarantee real ground penetration/contact force. -->
-        <collision>
+        <collision>
+            <!-- gazebo_ros_ackermann_drive auto-computes wheel radius from the
+                 collision shape but only supports cylinder/sphere primitives -
+                 an STL mesh collision here makes it silently use radius 0,
+                 which divides target_linear by zero and the car never drives.
+                 Use a cylinder sized to the wheel mesh (radius 0.033m) instead,
+                 keeping the STL for the visual only. -->
             <origin rpy="1.5708 0 0" xyz="0 0 0" />
             <geometry>
@@ -156,5 +157,5 @@
             <origin rpy="0 0 0" xyz="0 0 0" />
             <geometry>
-                <mesh filename="package://qcar_updated/models/qcar/QCarWheel.stl"
+                <mesh filename="file://$(find qcar_navigation)/meshes/QCarWheel.stl"
                     scale="0.001 0.001 0.001" />
             </geometry>
@@ -162,4 +163,10 @@
         </visual>
         <collision>
+            <!-- gazebo_ros_ackermann_drive auto-computes wheel radius from the
+                 collision shape but only supports cylinder/sphere primitives -
+                 an STL mesh collision here makes it silently use radius 0,
+                 which divides target_linear by zero and the car never drives.
+                 Use a cylinder sized to the wheel mesh (radius 0.033m) instead,
+                 keeping the STL for the visual only. -->
             <origin rpy="1.5708 0 0" xyz="0 0 0" />
             <geometry>
@@ -186,5 +193,5 @@
             <origin rpy="0 0 0" xyz="0 0 0" />
             <geometry>
-                <mesh filename="package://qcar_updated/models/qcar/QCarWheel.stl"
+                <mesh filename="file://$(find qcar_navigation)/meshes/QCarWheel.stl"
                     scale="0.001 0.001 0.001" />
             </geometry>
@@ -192,4 +199,10 @@
         </visual>
         <collision>
+            <!-- gazebo_ros_ackermann_drive auto-computes wheel radius from the
+                 collision shape but only supports cylinder/sphere primitives -
+                 an STL mesh collision here makes it silently use radius 0,
+                 which divides target_linear by zero and the car never drives.
+                 Use a cylinder sized to the wheel mesh (radius 0.033m) instead,
+                 keeping the STL for the visual only. -->
             <origin rpy="1.5708 0 0" xyz="0 0 0" />
             <geometry>
@@ -213,5 +226,5 @@
             <origin rpy="0 0 0" xyz="0 0 0" />
             <geometry>
-                <mesh filename="package://qcar_updated/models/qcar/QCarWheel.stl"
+                <mesh filename="file://$(find qcar_navigation)/meshes/QCarWheel.stl"
                     scale="0.001 0.001 0.001" />
             </geometry>
@@ -219,4 +232,10 @@
         </visual>
         <collision>
+            <!-- gazebo_ros_ackermann_drive auto-computes wheel radius from the
+                 collision shape but only supports cylinder/sphere primitives -
+                 an STL mesh collision here makes it silently use radius 0,
+                 which divides target_linear by zero and the car never drives.
+                 Use a cylinder sized to the wheel mesh (radius 0.033m) instead,
+                 keeping the STL for the visual only. -->
             <origin rpy="1.5708 0 0" xyz="0 0 0" />
             <geometry>
@@ -230,22 +249,4 @@
         </inertial>
     </link>
-    <!-- wheel-ground friction - without this the wheels spin freely with 100%
-         slip and the chassis never translates, regardless of PID gains -->
-    <gazebo reference="wheelfl">
-        <mu1>1.0</mu1>
-        <mu2>1.0</mu2>
-    </gazebo>
-    <gazebo reference="wheelfr">
-        <mu1>1.0</mu1>
-        <mu2>1.0</mu2>
-    </gazebo>
-    <gazebo reference="wheelrl">
-        <mu1>1.0</mu1>
-        <mu2>1.0</mu2>
-    </gazebo>
-    <gazebo reference="wheelrr">
-        <mu1>1.0</mu1>
-        <mu2>1.0</mu2>
-    </gazebo>
     <joint name="camera_rgb_joint" type="fixed">
         <!-- <axis xyz="0 1 0" /> -->
@@ -293,4 +294,25 @@
     </joint>
     <link name="camera_csi_left" />
+    <!-- Explicit high friction for the drive/steer wheels - without this the
+         ackermann plugin can spin the wheel joints at exactly the commanded
+         angular velocity (confirmed via debug logging) while the chassis
+         never actually translates, since URDF collisions get no friction
+         surface unless one is set here. -->
+    <gazebo reference="wheelfl">
+        <mu1>1.0</mu1>
+        <mu2>1.0</mu2>
+    </gazebo>
+    <gazebo reference="wheelfr">
+        <mu1>1.0</mu1>
+        <mu2>1.0</mu2>
+    </gazebo>
+    <gazebo reference="wheelrl">
+        <mu1>1.0</mu1>
+        <mu2>1.0</mu2>
+    </gazebo>
+    <gazebo reference="wheelrr">
+        <mu1>1.0</mu1>
+        <mu2>1.0</mu2>
+    </gazebo>
     <gazebo reference="camera_csi_front">
         <sensor type="camera" name="front_camera">
@@ -326,10 +348,12 @@
             <max_steer>0.5236</max_steer>
             <max_speed>20</max_speed>
-            <!-- PID tuning: the upstream demo's gains (1500/1000) were tuned for a
-                 full-size car and are ~1000x too aggressive for this vehicle's wheel
-                 inertia, causing an immediate physics blowup (confirmed by testing).
-                 0.3/0/0.02 steering gain still destabilized the sim (gzserver crash
-                 in Ogre::AxisAlignedBox::setExtents) even with the wheel inertia bump
-                 above - these lower values are confirmed stable. -->
+            <!-- PID tuning: this vehicle's wheel/steering-hub rotational inertia is tiny
+                 relative to a 100Hz control loop, so this is a genuinely stiff system -
+                 even modest P gains here can diverge (confirmed: wheel joint velocity
+                 goes NaN within ~1s at gain 1.0, and the resulting Ogre bounding-box
+                 assertion kills gzserver). These low gains are stability-verified and
+                 reach the commanded wheel speed within ~1s; retune upward with care and
+                 always verify gzserver survives a sustained forward command before
+                 trusting a new value. -->
             <left_steering_pid_gain>0.02 0 0.002</left_steering_pid_gain>
             <left_steering_i_range>0 0</left_steering_i_range>

Commit message: rpp in updated pkg

File: qcar_ackermann/urdf/qcar_model.xacro (robot description, xacro)
@@ -1,5 +1,5 @@
 <?xml version='1.0'?>
 <robot name="QCar" xmlns:xacro="http://www.ros.org/wiki/xacro">
-    <xacro:include filename="$(find qcar_ackermann)/urdf/materials.xacro" />
+  <xacro:include filename="$(find qcar_ackermann)/urdf/materials.xacro" />
     <link name="base">
         <visual>
@@ -116,5 +116,7 @@
         <child link="wheelfl" />
         <origin rpy="0 0 3.14" xyz="0 0 0" />
-        <axis xyz="0 1 0" />
+        <!-- axis negated to compensate for the 180deg yaw above (mesh mirror) -
+             without this the left wheel spins opposite the right wheel -->
+        <axis xyz="0 -1 0" />
     </joint>
     <link name="wheelfl">
@@ -127,9 +129,13 @@
             <material name="red" />
         </visual>
-        <collision>
-            <origin rpy="0 0 0" xyz="0 0 0" />
-            <geometry>
-                <mesh filename="package://qcar_ackermann/models/qcar/QCarWheel.stl"
-                    scale="0.001 0.001 0.001" />
+        <!-- collision is a cylinder, not the visual mesh - the ackermann drive
+             plugin's wheel-radius auto-detection only supports cylinder/sphere
+             collisions; with a mesh it silently reads radius=0 and poisons the
+             velocity PID. Radius is 3mm over the mesh's actual 0.033m to
+             guarantee real ground penetration/contact force. -->
+        <collision>
+            <origin rpy="1.5708 0 0" xyz="0 0 0" />
+            <geometry>
+                <cylinder radius="0.036" length="0.0245" />
             </geometry>
         </collision>
@@ -137,5 +143,5 @@
             <origin rpy="0 0 0" xyz="0 0 0" />
             <mass value="0.2" />
-            <inertia ixx="0.0000645" ixy="0" ixz="0" iyy="0.0001089" iyz="0" izz="0.0000645" />
+            <inertia ixx="0.0012" ixy="0" ixz="0" iyy="0.0022" iyz="0" izz="0.0012" />
         </inertial>
     </link>
@@ -156,8 +162,7 @@
         </visual>
         <collision>
-            <origin rpy="0 0 0" xyz="0 0 0" />
-            <geometry>
-                <mesh filename="package://qcar_ackermann/models/qcar/QCarWheel.stl"
-                    scale="0.001 0.001 0.001" />
+            <origin rpy="1.5708 0 0" xyz="0 0 0" />
+            <geometry>
+                <cylinder radius="0.036" length="0.0245" />
             </geometry>
         </collision>
@@ -165,5 +170,5 @@
             <origin rpy="0 0 0" xyz="0 0 0" />
             <mass value="0.2" />
-            <inertia ixx="0.0000645" ixy="0" ixz="0" iyy="0.0001089" iyz="0" izz="0.0000645" />
+            <inertia ixx="0.0012" ixy="0" ixz="0" iyy="0.0022" iyz="0" izz="0.0012" />
         </inertial>
     </link>
@@ -172,5 +177,8 @@
         <child link="wheelrl" />
         <origin rpy="0 0 3.14" xyz="-0.12765 0.05610 0.03338" />
-        <axis xyz="0 1 0" />
+        <!-- axis negated to compensate for the 180deg yaw above (mesh mirror) -
+             without this the left wheel spins opposite the right wheel for the
+             same signed velocity command -->
+        <axis xyz="0 -1 0" />
     </joint>
     <link name="wheelrl">
@@ -184,8 +192,7 @@
         </visual>
         <collision>
-            <origin rpy="0 0 0" xyz="0 0 0" />
-            <geometry>
-                <mesh filename="package://qcar_ackermann/models/qcar/QCarWheel.stl"
-                    scale="0.001 0.001 0.001" />
+            <origin rpy="1.5708 0 0" xyz="0 0 0" />
+            <geometry>
+                <cylinder radius="0.036" length="0.0245" />
             </geometry>
         </collision>
@@ -193,5 +200,5 @@
             <origin rpy="0 0 0" xyz="0 0 0" />
             <mass value="0.2" />
-            <inertia ixx="0.0000645" ixy="0" ixz="0" iyy="0.0001089" iyz="0" izz="0.0000645" />
+            <inertia ixx="0.0012" ixy="0" ixz="0" iyy="0.0022" iyz="0" izz="0.0012" />
         </inertial>
     </link>
@@ -212,8 +219,7 @@
         </visual>
         <collision>
-            <origin rpy="0 0 0" xyz="0 0 0" />
-            <geometry>
-                <mesh filename="package://qcar_ackermann/models/qcar/QCarWheel.stl"
-                    scale="0.001 0.001 0.001" />
+            <origin rpy="1.5708 0 0" xyz="0 0 0" />
+            <geometry>
+                <cylinder radius="0.036" length="0.0245" />
             </geometry>
         </collision>
@@ -221,7 +227,25 @@
             <origin rpy="0 0 0" xyz="0 0 0" />
             <mass value="0.2" />
-            <inertia ixx="0.0000645" ixy="0" ixz="0" iyy="0.0001089" iyz="0" izz="0.0000645" />
-        </inertial>
-    </link>
+            <inertia ixx="0.0012" ixy="0" ixz="0" iyy="0.0022" iyz="0" izz="0.0012" />
+        </inertial>
+    </link>
+    <!-- wheel-ground friction - without this the wheels spin freely with 100%
+         slip and the chassis never translates, regardless of PID gains -->
+    <gazebo reference="wheelfl">
+        <mu1>1.0</mu1>
+        <mu2>1.0</mu2>
+    </gazebo>
+    <gazebo reference="wheelfr">
+        <mu1>1.0</mu1>
+        <mu2>1.0</mu2>
+    </gazebo>
+    <gazebo reference="wheelrl">
+        <mu1>1.0</mu1>
+        <mu2>1.0</mu2>
+    </gazebo>
+    <gazebo reference="wheelrr">
+        <mu1>1.0</mu1>
+        <mu2>1.0</mu2>
+    </gazebo>
     <joint name="camera_rgb_joint" type="fixed">
         <!-- <axis xyz="0 1 0" /> -->
@@ -285,9 +309,46 @@
         </sensor>
     </gazebo>
+    <gazebo>
+        <plugin name="gazebo_ros_ackermann_drive" filename="libgazebo_ros_ackermann_drive.so">
+            <update_rate>100.0</update_rate>
+            <!-- front wheel spin joints (child of the steering hubs) -->
+            <front_left_joint>hubfl_wheelfl_joint</front_left_joint>
+            <front_right_joint>hubfr_wheelfr_joint</front_right_joint>
+            <!-- rear drive wheel joints -->
+            <rear_left_joint>base_wheelrl_joint</rear_left_joint>
+            <rear_right_joint>base_wheelrr_joint</rear_right_joint>
+            <!-- front hub steering (yaw) joints -->
+            <left_steering_joint>base_hubfl_joint</left_steering_joint>
+            <right_steering_joint>base_hubfr_joint</right_steering_joint>
+            <!-- wheelbase/track/wheel radius are auto-computed by the plugin
+                 from the joints' actual poses/collision geometry in this URDF -->
+            <!-- Real QCar steering limit: 30 deg -->
+            <max_steer>0.5236</max_steer>
+            <max_speed>20</max_speed>
+            <!-- PID tuning: the upstream demo's gains (1500/1000) were tuned for a
+                 full-size car and are ~1000x too aggressive for this vehicle's wheel
+                 inertia, causing an immediate physics blowup (confirmed by testing).
+                 0.3/0/0.02 steering gain still destabilized the sim (gzserver crash
+                 in Ogre::AxisAlignedBox::setExtents) even with the wheel inertia bump
+                 above - these lower values are confirmed stable. -->
+            <left_steering_pid_gain>3.0 0 0.1</left_steering_pid_gain>
+            <left_steering_i_range>0 0</left_steering_i_range>
+            <right_steering_pid_gain>3.0 0 0.1</right_steering_pid_gain>
+            <right_steering_i_range>0 0</right_steering_i_range>
+            <linear_velocity_pid_gain>0.3 0 0.005</linear_velocity_pid_gain>
+            <linear_velocity_i_range>0 0</linear_velocity_i_range>
+            <publish_odom>true</publish_odom>
+            <publish_odom_tf>true</publish_odom_tf>
+            <publish_wheel_tf>true</publish_wheel_tf>
+            <publish_distance>false</publish_distance>
+            <odometry_frame>odom</odometry_frame>
+            <robot_base_frame>base</robot_base_frame>
+        </plugin>
+    </gazebo>
     <!-- LiDAR Sensor -->
     <gazebo reference="lidar">
         <sensor type="ray" name="lidar_sensor">
             <pose>0 0 0 0 0 0</pose>
-            <visualize>false</visualize>
+            <visualize>true</visualize>
             <update_rate>10</update_rate>
             <ray>
@@ -320,37 +381,3 @@
         </sensor>
     </gazebo>
-    <!-- Ackermann drive plugin -->
-    <gazebo>
-        <plugin name="ackermann_drive" filename="libgazebo_ros_ackermann_drive.so">
-            <ros>
-                <namespace></namespace>
-            </ros>
-            <update_rate>100.0</update_rate>
-            <front_left_joint>hubfl_wheelfl_joint</front_left_joint>
-            <front_right_joint>hubfr_wheelfr_joint</front_right_joint>
-            <rear_left_joint>base_wheelrl_joint</rear_left_joint>
-            <rear_right_joint>base_wheelrr_joint</rear_right_joint>
-            <left_steering_joint>base_hubfl_joint</left_steering_joint>
-            <right_steering_joint>base_hubfr_joint</right_steering_joint>
-            <max_steer>0.5236</max_steer>
-            <max_steering_angle>0.5236</max_steering_angle>
-            <max_speed>3.0</max_speed>
-            <left_steering_pid_gain>5 0 0.1</left_steering_pid_gain>
-            <left_steering_i_range>0 0</left_steering_i_range>
-            <right_steering_pid_gain>5 0 0.1</right_steering_pid_gain>
-            <right_steering_i_range>0 0</right_steering_i_range>
-            <linear_velocity_pid_gain>10 0 0.5</linear_velocity_pid_gain>
-            <linear_velocity_i_range>0 0</linear_velocity_i_range>
-            <wheel_base>0.257</wheel_base>
-            <wheel_separation>0.112</wheel_separation>
-            <wheel_diameter>0.066</wheel_diameter>
-            <publish_odom>true</publish_odom>
-            <publish_odom_tf>true</publish_odom_tf>
-            <publish_wheel_tf>true</publish_wheel_tf>
-            <odometry_topic>odom</odometry_topic>
-            <odometry_frame>odom</odometry_frame>
-            <robot_base_frame>base</robot_base_frame>
-            <command_topic>cmd_vel</command_topic>
-        </plugin>
-    </gazebo>
-</robot>
+  </robot>
